File: hardware/aphid-direction-controller/MCU.kicad_sch (KiCad schematic)
At the start: 6 parts, among them J5 DEBUG, U1 STM32G431CBTx, Y1 16 MHz

Commit message: Worked on direction PCB
Parts:
- added C14, C15, C16, C17: 100nF, Capacitor_SMD:C_0603_1608Metric, symbol Device:C
- added R3: 10k, Resistor_SMD:R_0603_1608Metric, symbol Device:R
- renumbered C11 to C13, R11 to R4, U1 to U3
Connections:
- net +3.3V: now also J5.3 (VCC), U3.1 (VBAT), U3.24 (VDD), U3.36 (VDD), U3.48 (VDD), C14.1, C15.1, C17.1, R3.2
- net CAN_RX: now also U3.45 (PB8)
- net CAN_TX: now also U3.46 (PB9)
- net FORWARD_LIGHT: now also U3.8 (PA0)
- net FORWARD_PUSHED: now also U3.11 (PA3)
- net GND: now also J5.11 (GNDDetect), J5.5 (GND), J5.7 (GND), C14.2, C15.2, C16.2, C17.2
- net NEUTRAL_LIGHT: now also U3.9 (PA1)
- net NEUTRAL_PUSHED: now also U3.12 (PA4)
- net OSC_IN: now also U3.5 (PF0)
- net OSC_OUT: now also U3.6 (PF1)
- net REVERSE_LIGHT: now also U3.10 (PA2)
- net REVERSE_PUSHED: now also U3.13 (PA5)
- net VSENSE: now also U3.16 (PB0)
- net VDDA: now reaches U3.20 (VREF+)
- net VDDA: now also U3.21 (VDDA)
- net DBG_TX: now reaches U3.31 (PA9)
- net DBG_TX: now also J5.14 (VCP_TX)
- net DBG_RX: now reaches U3.32 (PA10)
- net DBG_RX: now also J5.13 (VCP_RX)
- net SWDIO: now reaches U3.37 (PA13)
- net SWDIO: now also J5.4 (JTMS/SWDIO)
- net SWCLK: now reaches U3.38 (PA14)
- net SWCLK: now also J5.6 (JCLK/SWCLK)
- net SWO: now reaches U3.40 (PB3)
- net SWO: now also J5.8 (JTDO/SWO)
- net NRST: now reaches U3.7 (PG10)
- net NRST: now also J5.12 (~{RST}), C16.1, R3.1
- no-connect marks 0 -> 23
Other:
- note added: "ADC1_IN15"
- note added: "FDCAN_RX (AF9)"
- note added: "FDCAN_TX (AF9)"
- note added: "PB8 is also BOOT0! Could add pull-down but I'll modify SWBOOT0 option byte instead"
- note added: "USART1_RX (AF7)"
- note added: "USART1_TX (AF7)"
- moved on the sheet: C12, C13, J5, R4, Y1
