File: hardware/aphid-direction-controller/aphid-direction-controller.kicad_pcb (KiCad board)
At the start: 2 copper layers, 65 parts, among them J1 FORWARD, J2 NEUTRAL, J3 REVERSE, J4 MAIN, J5 DEBUG, Q1 2N7002, Q2 2N7002, Q3 2N7002, U1 STM32G431CBTx, U2 TJA1042T-3, U3 LM78M05_TO252, U6 AMS1117-3.3, Y1 16 MHz

Commit message: Worked on direction PCB
Parts:
- added C14: 100nF, Capacitor_SMD:C_0603_1608Metric, F.Cu at (131.0, 89.8)
- added C15: 100nF, Capacitor_SMD:C_0603_1608Metric, F.Cu at (127.8, 99.2)
- added C16: 100nF, Capacitor_SMD:C_0603_1608Metric, F.Cu at (142.5, 77.2)
- added C17: 100nF, Capacitor_SMD:C_0603_1608Metric, F.Cu at (139.8, 91.0)
- added C8: 1uF, Capacitor_SMD:C_0603_1608Metric, F.Cu at (143.0, 95.0)
- added C9: 100nF, Capacitor_SMD:C_0603_1608Metric, F.Cu at (141.0, 95.0)
- added D7: PWR, LED_SMD:LED_0603_1608Metric, F.Cu at (119.2, 97.5)
- added FB1: 600, Inductor_SMD:L_0603_1608Metric, F.Cu at (145.0, 95.0)
- added R19: R, Resistor_SMD:R_0603_1608Metric, F.Cu at (119.2, 100.0)
- added R3: 10k, Resistor_SMD:R_0603_1608Metric, F.Cu at (142.5, 79.8)
- J1: footprint Connector_JST:JST_XH_B3B-XH-A_1x03_P2.50mm_Vertical -> Connector_JST:JST_PH_B4B-PH-K_1x04_P2.00mm_Vertical
- J2: renamed from J4; footprint Connector_JST:JST_XH_B4B-XH-A_1x04_P2.50mm_Vertical -> Connector_JST:JST_PH_B4B-PH-K_1x04_P2.00mm_Vertical
- J3: renamed from J2; footprint Connector_JST:JST_XH_B3B-XH-A_1x03_P2.50mm_Vertical -> Connector_JST:JST_PH_B4B-PH-K_1x04_P2.00mm_Vertical
- J4: renamed from J3; footprint Connector_JST:JST_XH_B3B-XH-A_1x03_P2.50mm_Vertical -> Connector_JST:JST_PH_B4B-PH-K_1x04_P2.00mm_Vertical
- moved J2 64.5 mm to (143.0, 130.6), turned to 180 degrees
- moved C27 58.1 mm to (155.0, 126.0)
- moved J4 52.5 mm to (160.6, 116.0), turned to -90 degrees
- moved D5 51.2 mm to (155.0, 119.0), turned to 180 degrees
- moved J3 48.8 mm to (160.6, 102.0), turned to -90 degrees
- moved H4 48.2 mm to (120.0, 130.0)
- moved H1 48.2 mm to (120.0, 80.0)
- moved C26 47.1 mm to (155.0, 112.0)
- moved J1 45.7 mm to (160.6, 88.0), turned to -90 degrees
- moved R11 42.3 mm to (155.0, 122.0), turned to 180 degrees
- moved R12 41.8 mm to (155.0, 124.0)
- moved Y1 41.1 mm to (133.0, 105.0), turned to 180 degrees
- moved C12 38.9 mm to (130.0, 105.0), turned to 90 degrees
- moved C13 36.7 mm to (136.0, 105.0), turned to -90 degrees
- moved C2 36.6 mm to (130.0, 125.0)
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- renumbered C28 to C1, C11 to C13, C4 to C18, C5 to C19, C9 to C2, C6 to C20, C18 to C21, C7 to C22, C8 to C23, C15 to C24, C10 to C25, C19 to C26, C20 to C27, C1 to C28, C2 to C29, C13 to C3, C3 to C30, C25 to C4, C16 to C5, C14 to C6, C17 to C7, D5 to D2, D4 to D3, D3 to D4, D2 to D5, L4 to L1, L1 to L2, R18 to R1, R13 to R10, R14 to R11, R15 to R12, R2 to R13, R3 to R14, R5 to R15, R1 to R16, R4 to R17, R6 to R18, R19 to R2, R11 to R4, R7 to R5, R8 to R6, R9 to R7, R10 to R8, R12 to R9, U3 to U1, U6 to U2, U1 to U3, U2 to U4
Connections:
- J2 pad 1: GND -> /CAN/CANH
- J2 pad 2: /Connectors/VIN -> /CAN/CANL
- J2 pad 3: /CAN/CANL -> /Connectors/VIN
- J2 pad 4: /CAN/CANH -> GND
- J5 pad 11: unconnected-(J5-GNDDetect-Pad11) -> GND
- J5 pad 12: unconnected-(J5-~{RST}-Pad12) -> /MCU/NRST
- J5 pad 13: unconnected-(J5-VCP_RX-Pad13) -> /MCU/DBG_RX
- J5 pad 14: unconnected-(J5-VCP_TX-Pad14) -> /MCU/DBG_TX
- J5 pad 3: unconnected-(J5-VCC-Pad3) -> +3.3V
- J5 pad 4: unconnected-(J5-JTMS/SWDIO-Pad4) -> /MCU/SWDIO
- J5 pad 5: Net-(J5-GND-Pad5) -> GND
- J5 pad 6: unconnected-(J5-JCLK/SWCLK-Pad6) -> /MCU/SWCLK
- J5 pad 7: Net-(J5-GND-Pad5) -> GND
- J5 pad 8: unconnected-(J5-JTDO/SWO-Pad8) -> /MCU/SWO
- R1 pad 1: /MCU/VSENSE -> +12V
- R1 pad 2: /Connectors/VIN -> /MCU/VSENSE
- U3 pad 1: unconnected-(U1-VBAT-Pad1) -> +3.3V
- U3 pad 10: unconnected-(U1-PA2-Pad10) -> /LEDs/REVERSE_LIGHT
- U3 pad 11: unconnected-(U1-PA3-Pad11) -> /Buttons/FORWARD_PUSHED
- U3 pad 12: unconnected-(U1-PA4-Pad12) -> /Buttons/NEUTRAL_PUSHED
- U3 pad 13: unconnected-(U1-PA5-Pad13) -> /Buttons/REVERSE_PUSHED
- U3 pad 16: unconnected-(U1-PB0-Pad16) -> /MCU/VSENSE
- U3 pad 20: unconnected-(U1-VREF+-Pad20) -> VDDA
- U3 pad 21: unconnected-(U1-VDDA-Pad21) -> VDDA
- U3 pad 24: unconnected-(U1-VDD-Pad24) -> +3.3V
- U3 pad 31: unconnected-(U1-PA9-Pad31) -> /MCU/DBG_TX
- U3 pad 32: unconnected-(U1-PA10-Pad32) -> /MCU/DBG_RX
- U3 pad 36: unconnected-(U1-VDD-Pad36) -> +3.3V
- U3 pad 37: unconnected-(U1-PA13-Pad37) -> /MCU/SWDIO
- U3 pad 38: unconnected-(U1-PA14-Pad38) -> /MCU/SWCLK
- U3 pad 40: unconnected-(U1-PB3-Pad40) -> /MCU/SWO
- U3 pad 45: unconnected-(U1-PB8-Pad45) -> /CAN/CAN_RX
- U3 pad 46: unconnected-(U1-PB9-Pad46) -> /CAN/CAN_TX
- U3 pad 48: unconnected-(U1-VDD-Pad48) -> +3.3V
- U3 pad 5: unconnected-(U1-PF0-Pad5) -> /MCU/OSC_IN
- U3 pad 6: unconnected-(U1-PF1-Pad6) -> /MCU/OSC_OUT
- U3 pad 7: unconnected-(U1-PG10-Pad7) -> /MCU/NRST
- U3 pad 8: unconnected-(U1-PA0-Pad8) -> /LEDs/FORWARD_LIGHT
- U3 pad 9: unconnected-(U1-PA1-Pad9) -> /LEDs/NEUTRAL_LIGHT
Routing:
- net /Connectors/FORWARD_LED: track 0.00 -> 10.7 mm
- net /Buttons/FORWARD_BUTTON: track 0.00 -> 6.55 mm
- net /Buttons/FORWARD_PUSHED: track 0.00 -> 4.02 mm
- net Net-(Q1-D): track 0.00 -> 2.42 mm
- net GND: vias 0 -> 30
- added copper zone on In2.Cu, net +3.3V
- added copper zone on In1.Cu, net GND
Other:
- board outline added: 50 x 60 mm
- copper layers 2 -> 4
