File: hardware/aphid-direction-controller/can.kicad_sch (KiCad schematic)
At the start: 13 parts, among them U2 TJA1042T-3

Commit message: Worked on direction PCB
Parts:
- renumbered C4 to C18, C5 to C19, C6 to C20, C18 to C21, C7 to C22, C8 to C23, C15 to C24, L1 to L2, R7 to R5, R8 to R6, U2 to U4
Changed lines of the file:
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@@
 		(dnp no)
 		(fields_autoplaced yes)
-		(property "Reference" "#PWR037"
+		(property "Reference" "#PWR060"
 			(at 170.18 102.87 0)
 			(effects
@@
 			(project "aphid-direction-controller"
 				(path "/08e61dba-ec41-4bf0-9be1-028614d183d2/c08ed64c-2d0d-4120-bd88-c312a29aa4b5"
-					(reference "#PWR037")
+					(reference "#PWR060")
 					(unit 1)
 				)
@@
 		(dnp no)
 		(fields_autoplaced yes)
-		(property "Reference" "C4"
+		(property "Reference" "C18"
 			(at 46.99 34.2899 0)
 			(effects
@@
 			(project "aphid-direction-controller"
 				(path "/08e61dba-ec41-4bf0-9be1-028614d183d2/c08ed64c-2d0d-4120-bd88-c312a29aa4b5"
-					(reference "C4")
+					(reference "C18")
 					(unit 1)
 				)
@@
 		(dnp no)
 		(fields_autoplaced yes)
-		(property "Reference" "#PWR034"
+		(property "Reference" "#PWR055"
 			(at 110.49 102.87 0)
 			(effects
@@
 			(project "aphid-direction-controller"
 				(path "/08e61dba-ec41-4bf0-9be1-028614d183d2/c08ed64c-2d0d-4120-bd88-c312a29aa4b5"
-					(reference "#PWR034")
+					(reference "#PWR055")
 					(unit 1)
 				)
@@
 		(dnp no)
 		(fields_autoplaced yes)
-		(property "Reference" "L1"
+		(property "Reference" "L2"
 			(at 187.706 71.12 0)
 			(effects
@@
 			(project "aphid-direction-controller"
 				(path "/08e61dba-ec41-4bf0-9be1-028614d183d2/c08ed64c-2d0d-4120-bd88-c312a29aa4b5"
-					(reference "L1")
+					(reference "L2")
 					(unit 1)
 				)
@@
 		(dnp no)
 		(fields_autoplaced yes)
-		(property "Reference" "R8"
+		(property "Reference" "R6"
 			(at 215.9 96.5199 0)
 			(effects
@@
 			(project "aphid-direction-controller"
 				(path "/08e61dba-ec41-4bf0-9be1-028614d183d2/c08ed64c-2d0d-4120-bd88-c312a29aa4b5"
-					(reference "R8")
+					(reference "R6")
 					(unit 1)
 				)
@@
 		(dnp no)
 		(fields_autoplaced yes)
-		(property "Reference" "#PWR035"
+		(property "Reference" "#PWR058"
 			(at 143.51 102.87 0)
 			(effects
@@
 			(project "aphid-direction-controller"
 				(path "/08e61dba-ec41-4bf0-9be1-028614d183d2/c08ed64c-2d0d-4120-bd88-c312a29aa4b5"
-					(reference "#PWR035")
+					(reference "#PWR058")
 					(unit 1)
 				)
@@
 		(dnp no)
 		(fields_autoplaced yes)
-		(property "Reference" "#PWR036"
+		(property "Reference" "#PWR059"
 			(at 157.48 102.87 0)
 			(effects
@@
 			(project "aphid-direction-controller"
 				(path "/08e61dba-ec41-4bf0-9be1-028614d183d2/c08ed64c-2d0d-4120-bd88-c312a29aa4b5"
-					(reference "#PWR036")
+					(reference "#PWR059")
 					(unit 1)
 				)
@@
 		(dnp no)
 		(fields_autoplaced yes)
-		(property "Reference" "C5"
+		(property "Reference" "C19"
 			(at 59.69 34.2899 0)
 			(effects
@@
 			(project "aphid-direction-controller"
 				(path "/08e61dba-ec41-4bf0-9be1-028614d183d2/c08ed64c-2d0d-4120-bd88-c312a29aa4b5"
-					(reference "C5")
+					(reference "C19")
 					(unit 1)
 				)
@@
 		(dnp no)
 		(fields_autoplaced yes)
-		(property "Reference" "#PWR025"
+		(property "Reference" "#PWR051"
 			(at 43.18 48.26 0)
 			(effects
@@
 			(project "aphid-direction-controller"
 				(path "/08e61dba-ec41-4bf0-9be1-028614d183d2/c08ed64c-2d0d-4120-bd88-c312a29aa4b5"
-					(reference "#PWR025")
+					(reference "#PWR051")
 					(unit 1)
 				)
@@
 		(dnp no)
 		(fields_autoplaced yes)
-		(property "Reference" "C18"
+		(property "Reference" "C21"
 			(at 173.99 87.6299 0)
 			(effects
@@
 			(project "aphid-direction-controller"
 				(path "/08e61dba-ec41-4bf0-9be1-028614d183d2/c08ed64c-2d0d-4120-bd88-c312a29aa4b5"
-					(reference "C18")
+					(reference "C21")
 					(unit 1)
 				)
@@
 		(on_board yes)
 		(dnp no)
-		(property "Reference" "C7"
+		(property "Reference" "C22"
 			(at 176.53 77.4762 0)
 			(effects
@@
 			(project "aphid-direction-controller"
 				(path "/08e61dba-ec41-4bf0-9be1-028614d183d2/c08ed64c-2d0d-4120-bd88-c312a29aa4b5"
-					(reference "C7")
+					(reference "C22")
 					(unit 1)
 				)
@@
 		(dnp no)
 		(fields_autoplaced yes)
-		(property "Reference" "C15"
+		(property "Reference" "C24"
 			(at 214.63 109.2199 0)
 			(effects
@@
 			(project "aphid-direction-controller"
 				(path "/08e61dba-ec41-4bf0-9be1-028614d183d2/c08ed64c-2d0d-4120-bd88-c312a29aa4b5"
-					(reference "C15")
+					(reference "C24")
 					(unit 1)
 				)
@@
 		(dnp no)
 		(fields_autoplaced yes)
-		(property "Reference" "#PWR033"
+		(property "Reference" "#PWR061"
 			(at 210.82 123.19 0)
 			(effects
@@
 			(project "aphid-direction-controller"
 				(path "/08e61dba-ec41-4bf0-9be1-028614d183d2/c08ed64c-2d0d-4120-bd88-c312a29aa4b5"
-					(reference "#PWR033")
+					(reference "#PWR061")
 					(unit 1)
 				)
@@
 		(on_board yes)
 		(dnp no)
-		(property "Reference" "R7"
+		(property "Reference" "R5"
 			(at 205.74 96.5199 0)
 			(effects
@@
 			(project "aphid-direction-controller"
 				(path "/08e61dba-ec41-4bf0-9be1-028614d183d2/c08ed64c-2d0d-4120-bd88-c312a29aa4b5"
-					(reference "R7")
+					(reference "R5")
 					(unit 1)
 				)
@@
 		(dnp no)
 		(fields_autoplaced yes)
-		(property "Reference" "#PWR03"
+		(property "Reference" "#PWR054"
 			(at 114.3 81.28 0)
 			(effects
@@
 			(project "aphid-direction-controller"
 				(path "/08e61dba-ec41-4bf0-9be1-028614d183d2/c08ed64c-2d0d-4120-bd88-c312a29aa4b5"
-					(reference "#PWR03")
+					(reference "#PWR054")
 					(unit 1)
 				)
@@
 		(dnp no)
 		(fields_autoplaced yes)
-		(property "Reference" "#PWR023"
+		(property "Reference" "#PWR050"
 			(at 43.18 33.02 0)
 			(effects
@@
 			(project "aphid-direction-controller"
 				(path "/08e61dba-ec41-4bf0-9be1-028614d183d2/c08ed64c-2d0d-4120-bd88-c312a29aa4b5"
-					(reference "#PWR023")
+					(reference "#PWR050")
 					(unit 1)
 				)
@@
 			)
 		)
-		(property "Datasheet" "http://www.onsemi.com/pub_link/Collateral/NUP2105L-D.PDF"
+		(property "Datasheet" "https://www.onsemi.com/pub_link/Collateral/NUP2105L-D.PDF"
 			(at 146.685 85.725 0)
 			(effects
@@
 		(dnp no)
 		(fields_autoplaced yes)
-		(property "Reference" "C6"
+		(property "Reference" "C20"
 			(at 161.29 87.6299 0)
 			(effects
@@
 			(project "aphid-direction-controller"
 				(path "/08e61dba-ec41-4bf0-9be1-028614d183d2/c08ed64c-2d0d-4120-bd88-c312a29aa4b5"
-					(reference "C6")
+					(reference "C20")
 					(unit 1)
 				)
@@
 		(dnp no)
 		(fields_autoplaced yes)
-		(property "Reference" "#PWR024"
+		(property "Reference" "#PWR052"
 			(at 55.88 33.02 0)
 			(effects
@@
 			(project "aphid-direction-controller"
 				(path "/08e61dba-ec41-4bf0-9be1-028614d183d2/c08ed64c-2d0d-4120-bd88-c312a29aa4b5"
-					(reference "#PWR024")
+					(reference "#PWR052")
 					(unit 1)
 				)
@@
 		(on_board yes)
 		(dnp no)
-		(property "Reference" "C8"
+		(property "Reference" "C23"
 			(at 199.39 77.4762 0)
 			(effects
@@
 			(project "aphid-direction-controller"
 				(path "/08e61dba-ec41-4bf0-9be1-028614d183d2/c08ed64c-2d0d-4120-bd88-c312a29aa4b5"
-					(reference "C8")
+					(reference "C23")
 					(unit 1)
 				)
@@
 		(dnp no)
 		(fields_autoplaced yes)
-		(property "Reference" "#PWR026"
+		(property "Reference" "#PWR053"
 			(at 55.88 48.26 0)
 			(effects
@@
 			(project "aphid-direction-controller"
 				(path "/08e61dba-ec41-4bf0-9be1-028614d183d2/c08ed64c-2d0d-4120-bd88-c312a29aa4b5"
-					(reference "#PWR026")
+					(reference "#PWR053")
 					(unit 1)
 				)
@@
 		(dnp no)
 		(fields_autoplaced yes)
-		(property "Reference" "#PWR01"
+		(property "Reference" "#PWR056"
 			(at 125.73 69.85 0)
 			(effects
@@
 			(project "aphid-direction-controller"
 				(path "/08e61dba-ec41-4bf0-9be1-028614d183d2/c08ed64c-2d0d-4120-bd88-c312a29aa4b5"
-					(reference "#PWR01")
+					(reference "#PWR056")
 					(unit 1)
 				)
@@
 		(dnp no)
 		(fields_autoplaced yes)
-		(property "Reference" "#PWR02"
+		(property "Reference" "#PWR057"
 			(at 125.73 102.87 0)
 			(effects
@@
 			(project "aphid-direction-controller"
 				(path "/08e61dba-ec41-4bf0-9be1-028614d183d2/c08ed64c-2d0d-4120-bd88-c312a29aa4b5"
-					(reference "#PWR02")
+					(reference "#PWR057")
 					(unit 1)
 				)
@@
 		(dnp no)
 		(fields_autoplaced yes)
-		(property "Reference" "U2"
+		(property "Reference" "U4"
 			(at 127.9241 66.04 0)
 			(effects
@@
 			(project "aphid-direction-controller"
 				(path "/08e61dba-ec41-4bf0-9be1-028614d183d2/c08ed64c-2d0d-4120-bd88-c312a29aa4b5"
-					(reference "U2")
-					(unit 1)
-				)
+					(reference "U4")
+					(unit 1)
+				)
