File: hardware/aphid-direction-controller/connectors.kicad_sch (KiCad schematic)
At the start: 7 parts, among them J1 FORWARD, J2 NEUTRAL, J3 REVERSE, J4 MAIN

Commit message: Worked on direction PCB
Parts:
- J1: footprint Connector_JST:JST_XH_B3B-XH-A_1x03_P2.50mm_Vertical -> Connector_JST:JST_PH_B4B-PH-K_1x04_P2.00mm_Vertical; symbol Connector_Generic:Conn_01x03 -> Connector_Generic:Conn_01x04
- J2: renamed from J4; footprint Connector_JST:JST_XH_B4B-XH-A_1x04_P2.50mm_Vertical -> Connector_JST:JST_PH_B4B-PH-K_1x04_P2.00mm_Vertical
- J3: renamed from J2; footprint Connector_JST:JST_XH_B3B-XH-A_1x03_P2.50mm_Vertical -> Connector_JST:JST_PH_B4B-PH-K_1x04_P2.00mm_Vertical; symbol Connector_Generic:Conn_01x03 -> Connector_Generic:Conn_01x04
- J4: renamed from J3; footprint Connector_JST:JST_XH_B3B-XH-A_1x03_P2.50mm_Vertical -> Connector_JST:JST_PH_B4B-PH-K_1x04_P2.00mm_Vertical; symbol Connector_Generic:Conn_01x03 -> Connector_Generic:Conn_01x04
- renumbered D4 to D3, D3 to D4, D2 to D5
Connections:
- net +5V: now also J1.4 (Pin_4), J3.4 (Pin_4), J4.4 (Pin_4)
- net CANH: now also J2.1 (Pin_1); no longer J2.4 (Pin_4)
- net CANL: now also J2.2 (Pin_2); no longer J2.3 (Pin_3)
- net GND: now also J2.4 (Pin_4); no longer J2.1 (Pin_1)
- net VIN: now also J2.3 (Pin_3); no longer J2.2 (Pin_2)
