File: hardware/aphid-direction-controller/leds.kicad_sch (KiCad schematic)
At the start: 12 parts, among them Q1 2N7002, Q2 2N7002, Q3 2N7002

Commit message: Worked on direction PCB
Parts:
- renumbered C1 to C28, C2 to C29, C3 to C30, R2 to R13, R3 to R14, R5 to R15, R1 to R16, R4 to R17, R6 to R18
Changed lines of the file:
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@@
 		(dnp no)
 		(fields_autoplaced yes)
-		(property "Reference" "#PWR015"
+		(property "Reference" "#PWR068"
 			(at 115.57 85.09 0)
 			(effects
@@
 			(project "aphid-direction-controller"
 				(path "/08e61dba-ec41-4bf0-9be1-028614d183d2/e7d5e156-c64e-4541-9faa-542d2ea4ca82"
-					(reference "#PWR015")
+					(reference "#PWR068")
 					(unit 1)
 				)
@@
 		(dnp no)
 		(fields_autoplaced yes)
-		(property "Reference" "C3"
+		(property "Reference" "C30"
 			(at 146.05 134.6199 0)
 			(effects
@@
 			(project "aphid-direction-controller"
 				(path "/08e61dba-ec41-4bf0-9be1-028614d183d2/e7d5e156-c64e-4541-9faa-542d2ea4ca82"
-					(reference "C3")
+					(reference "C30")
 					(unit 1)
 				)
@@
 		(dnp no)
 		(fields_autoplaced yes)
-		(property "Reference" "#PWR022"
+		(property "Reference" "#PWR076"
 			(at 142.24 148.59 0)
 			(effects
@@
 			(project "aphid-direction-controller"
 				(path "/08e61dba-ec41-4bf0-9be1-028614d183d2/e7d5e156-c64e-4541-9faa-542d2ea4ca82"
-					(reference "#PWR022")
+					(reference "#PWR076")
 					(unit 1)
 				)
@@
 		(dnp no)
 		(fields_autoplaced yes)
-		(property "Reference" "R4"
+		(property "Reference" "R17"
 			(at 128.27 93.9799 0)
 			(effects
@@
 			(project "aphid-direction-controller"
 				(path "/08e61dba-ec41-4bf0-9be1-028614d183d2/e7d5e156-c64e-4541-9faa-542d2ea4ca82"
-					(reference "R4")
+					(reference "R17")
 					(unit 1)
 				)
@@
 		(dnp no)
 		(fields_autoplaced yes)
-		(property "Reference" "#PWR018"
+		(property "Reference" "#PWR072"
 			(at 125.73 125.73 0)
 			(effects
@@
 			(project "aphid-direction-controller"
 				(path "/08e61dba-ec41-4bf0-9be1-028614d183d2/e7d5e156-c64e-4541-9faa-542d2ea4ca82"
-					(reference "#PWR018")
+					(reference "#PWR072")
 					(unit 1)
 				)
@@
 		(dnp no)
 		(fields_autoplaced yes)
-		(property "Reference" "#PWR020"
+		(property "Reference" "#PWR070"
 			(at 115.57 166.37 0)
 			(effects
@@
 			(project "aphid-direction-controller"
 				(path "/08e61dba-ec41-4bf0-9be1-028614d183d2/e7d5e156-c64e-4541-9faa-542d2ea4ca82"
-					(reference "#PWR020")
+					(reference "#PWR070")
 					(unit 1)
 				)
@@
 		(dnp no)
 		(fields_autoplaced yes)
-		(property "Reference" "#PWR017"
+		(property "Reference" "#PWR069"
 			(at 115.57 125.73 0)
 			(effects
@@
 			(project "aphid-direction-controller"
 				(path "/08e61dba-ec41-4bf0-9be1-028614d183d2/e7d5e156-c64e-4541-9faa-542d2ea4ca82"
-					(reference "#PWR017")
+					(reference "#PWR069")
 					(unit 1)
 				)
@@
 		(dnp no)
 		(fields_autoplaced yes)
-		(property "Reference" "C2"
+		(property "Reference" "C29"
 			(at 146.05 93.9799 0)
 			(effects
@@
 			(project "aphid-direction-controller"
 				(path "/08e61dba-ec41-4bf0-9be1-028614d183d2/e7d5e156-c64e-4541-9faa-542d2ea4ca82"
-					(reference "C2")
+					(reference "C29")
 					(unit 1)
 				)
@@
 		(dnp no)
 		(fields_autoplaced yes)
-		(property "Reference" "#PWR021"
+		(property "Reference" "#PWR073"
 			(at 125.73 166.37 0)
 			(effects
@@
 			(project "aphid-direction-controller"
 				(path "/08e61dba-ec41-4bf0-9be1-028614d183d2/e7d5e156-c64e-4541-9faa-542d2ea4ca82"
-					(reference "#PWR021")
+					(reference "#PWR073")
 					(unit 1)
 				)
@@
 		(dnp no)
 		(fields_autoplaced yes)
-		(property "Reference" "#PWR014"
+		(property "Reference" "#PWR074"
 			(at 142.24 67.31 0)
 			(effects
@@
 			(project "aphid-direction-controller"
 				(path "/08e61dba-ec41-4bf0-9be1-028614d183d2/e7d5e156-c64e-4541-9faa-542d2ea4ca82"
-					(reference "#PWR014")
+					(reference "#PWR074")
 					(unit 1)
 				)
@@
 		(on_board yes)
 		(dnp no)
-		(property "Reference" "R5"
+		(property "Reference" "R15"
 			(at 118.11 152.3999 0)
 			(effects
@@
 			(project "aphid-direction-controller"
 				(path "/08e61dba-ec41-4bf0-9be1-028614d183d2/e7d5e156-c64e-4541-9faa-542d2ea4ca82"
-					(reference "R5")
+					(reference "R15")
 					(unit 1)
 				)
@@
 		(dnp no)
 		(fields_autoplaced yes)
-		(property "Reference" "R6"
+		(property "Reference" "R18"
 			(at 128.27 134.6199 0)
 			(effects
@@
 			(project "aphid-direction-controller"
 				(path "/08e61dba-ec41-4bf0-9be1-028614d183d2/e7d5e156-c64e-4541-9faa-542d2ea4ca82"
-					(reference "R6")
+					(reference "R18")
 					(unit 1)
 				)
@@
 		(on_board yes)
 		(dnp no)
-		(property "Reference" "R2"
+		(property "Reference" "R13"
 			(at 118.11 71.1199 0)
 			(effects
@@
 			(project "aphid-direction-controller"
 				(path "/08e61dba-ec41-4bf0-9be1-028614d183d2/e7d5e156-c64e-4541-9faa-542d2ea4ca82"
-					(reference "R2")
+					(reference "R13")
 					(unit 1)
 				)
@@
 		(dnp no)
 		(fields_autoplaced yes)
-		(property "Reference" "R1"
+		(property "Reference" "R16"
 			(at 128.27 53.3399 0)
 			(effects
@@
 			(project "aphid-direction-controller"
 				(path "/08e61dba-ec41-4bf0-9be1-028614d183d2/e7d5e156-c64e-4541-9faa-542d2ea4ca82"
-					(reference "R1")
+					(reference "R16")
 					(unit 1)
 				)
@@
 		(dnp no)
 		(fields_autoplaced yes)
-		(property "Reference" "C1"
+		(property "Reference" "C28"
 			(at 146.05 53.3399 0)
 			(effects
@@
 			(project "aphid-direction-controller"
 				(path "/08e61dba-ec41-4bf0-9be1-028614d183d2/e7d5e156-c64e-4541-9faa-542d2ea4ca82"
-					(reference "C1")
+					(reference "C28")
 					(unit 1)
 				)
@@
 		(dnp no)
 		(fields_autoplaced yes)
-		(property "Reference" "#PWR019"
+		(property "Reference" "#PWR075"
 			(at 142.24 107.95 0)
 			(effects
@@
 			(project "aphid-direction-controller"
 				(path "/08e61dba-ec41-4bf0-9be1-028614d183d2/e7d5e156-c64e-4541-9faa-542d2ea4ca82"
-					(reference "#PWR019")
+					(reference "#PWR075")
 					(unit 1)
 				)
@@
 		(dnp no)
 		(fields_autoplaced yes)
-		(property "Reference" "#PWR016"
+		(property "Reference" "#PWR071"
 			(at 125.73 85.09 0)
 			(effects
@@
 			(project "aphid-direction-controller"
 				(path "/08e61dba-ec41-4bf0-9be1-028614d183d2/e7d5e156-c64e-4541-9faa-542d2ea4ca82"
-					(reference "#PWR016")
+					(reference "#PWR071")
 					(unit 1)
 				)
@@
 		(on_board yes)
 		(dnp no)
-		(property "Reference" "R3"
+		(property "Reference" "R14"
 			(at 118.11 111.7599 0)
 			(effects
@@
 			(project "aphid-direction-controller"
 				(path "/08e61dba-ec41-4bf0-9be1-028614d183d2/e7d5e156-c64e-4541-9faa-542d2ea4ca82"
-					(reference "R3")
-					(unit 1)
-				)
+					(reference "R14")
+					(unit 1)
+				)
