File: hardware/aphid-direction-controller/power.kicad_sch (KiCad schematic)
At the start: 14 parts, among them U3 LM78M05_TO252, U6 AMS1117-3.3

Commit message: Worked on direction PCB
Parts:
- added C8: 1uF, Capacitor_SMD:C_0603_1608Metric, symbol Device:C
- added C9: 100nF, Capacitor_SMD:C_0603_1608Metric, symbol Device:C
- added D7: PWR, LED_SMD:LED_0603_1608Metric, symbol Device:LED
- added FB1: 600, Inductor_SMD:L_0603_1608Metric, symbol Device:FerriteBead_Small
- added R19: R, Resistor_SMD:R_0603_1608Metric, symbol Device:R
- renumbered C28 to C1, C9 to C2, C13 to C3, C25 to C4, C16 to C5, C14 to C6, C17 to C7, D5 to D2, L4 to L1, R18 to R1, R19 to R2, U3 to U1, U6 to U2
Connections:
- net +12V: now also R1.1
- net +3.3V: now also FB1.1, R19.1
- net GND: now also C8.2, C9.2, D7.1 (K)
- net VIN: no longer R1.2
- net VSENSE: now also R1.2; no longer R1.1
- new net: D7.2 (A), R19.2
- new net VDDA: C8.1, C9.1, FB1.2
Other:
- moved on the sheet: C4, D1, D2, L1, R1, R2
