File: hardware/aphid-bms-master/slave_power.kicad_sch (KiCad schematic)
At the start: 3 parts, among them Q1 ZXMP4A16G

Commit message: Assigned some footprints
Parts:
- C1: footprint (none) -> Capacitor_SMD:C_0805_2012Metric
- R2: footprint (none) -> Resistor_SMD:R_0805_2012Metric
Changed lines of the file:
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@@
 			)
 		)
-		(property "Footprint" ""
+		(property "Footprint" "Capacitor_SMD:C_0805_2012Metric"
 			(at 150.8252 85.09 0)
 			(effects
@@
 			)
 		)
-		(property "Footprint" ""
+		(property "Footprint" "Resistor_SMD:R_0805_2012Metric"
 			(at 143.51 64.262 90)
 			(effects

Commit message: Worked on BMS master
Parts:
- C1: footprint Capacitor_SMD:C_0805_2012Metric -> Capacitor_SMD:C_0603_1608Metric
Other:
- company: (none) -> https://aphid-ev.se
- title: (none) -> Aphid BMS Master
Changed lines of the file:
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@@
 	(generator_version "8.0")
 	(paper "A4")
+	(title_block
+		(title "Aphid BMS Master")
+		(date "2024-07-06")
+		(rev "1.0")
+		(company "https://aphid-ev.se")
+	)
 	(junction
 		(at 149.86 66.04)
@@
 			)
 		)
-		(property "Footprint" "Capacitor_SMD:C_0805_2012Metric"
+		(property "Footprint" "Capacitor_SMD:C_0603_1608Metric"
 			(at 150.8252 85.09 0)
 			(effects

Commit message: Worked on BMS master layout
Parts:
- C1: footprint Capacitor_SMD:C_0603_1608Metric -> Capacitor_SMD:C_0805_2012Metric
Changed lines of the file:
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@@
 			)
 		)
-		(property "Footprint" "Capacitor_SMD:C_0603_1608Metric"
+		(property "Footprint" "Capacitor_SMD:C_0805_2012Metric"
 			(at 150.8252 85.09 0)
 			(effects
