File: hardware/aphid-bms-master/aphid-bms-master.kicad_pcb (KiCad board)
At the start: 4 copper layers, 73 parts, among them J1 Main, J2 Slaves, J3 ContactorPos, J4 ContactorNeg, J5 ContactorPrecharge, J6 DEBUG, Q1 ZXMP4A16G, U1 STM32G491CCTx, U2 TJA1042T-3, U3 TJA1042T-3, U4 LMR33620BDDA, U5 LD1117S33, U6 DRV8803, Y1 8 MHz

Commit message: Worked on BMS master layout
Parts:
- C1: footprint Capacitor_SMD:C_0603_1608Metric -> Capacitor_SMD:C_0805_2012Metric
- D3, D4: footprint Diode_SMD:D_SOD-123 -> Diode_SMD:D_SMC
- U6: footprint Package_SO:SOIC-16W_7.5x12.8mm_P1.27mm -> Package_SO:SOIC-20W_7.5x12.8mm_P1.27mm
- moved J2 128.2 mm to (95.0, 148.9), turned to 180 degrees
- moved H3 127.7 mm to (161.0, 150.5)
- moved R1 117.7 mm to (90.0, 139.0)
- moved H2 115.5 mm to (161.0, 98.0)
- moved L2 109.9 mm to (93.5, 138.0), turned to -90 degrees
- moved JP1 106.6 mm to (175.7, 136.4)
- moved R9 106.6 mm to (175.7, 133.2)
- moved JP3 106.6 mm to (162.2, 116.0)
- moved D2 102.8 mm to (93.5, 132.5), turned to 90 degrees
- moved C23 97.7 mm to (91.0, 132.0), turned to -90 degrees
- moved C25 94.9 mm to (93.5, 122.0)
- moved U3 94.8 mm to (93.5, 126.5), turned to -90 degrees
- moved R2 84.7 mm to (84.5, 127.0)
- moved Q1 84.2 mm to (84.5, 132.5), turned to -90 degrees
- moved C1 80.2 mm to (84.5, 125.0), turned to 180 degrees
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
Commit message: Worked on BMS master layout
Parts:
- C14: footprint Capacitor_SMD:C_0603_1608Metric -> Capacitor_SMD:C_0805_2012Metric
- C2, C3, C9: footprint Capacitor_SMD:C_0805_2012Metric -> Capacitor_SMD:C_0603_1608Metric
- H1, H2, H3, H4: footprint MountingHole:MountingHole_3.2mm_M3 -> MountingHole:MountingHole_4.3mm_M4
- moved JP1 75.0 mm to (236.2, 92.0)
- moved R8 53.7 mm to (182.0, 74.0)
- moved FB1 52.6 mm to (151.5, 105.5)
- moved C19 51.2 mm to (149.5, 116.0), turned to 90 degrees
- moved C3 50.8 mm to (166.5, 112.0), turned to -90 degrees
- moved C17 49.0 mm to (155.5, 105.5)
- moved C18 48.8 mm to (155.5, 107.5)
- moved C2 48.5 mm to (166.5, 116.0), turned to 90 degrees
- moved C20 48.4 mm to (152.5, 107.5)
- moved Y1 42.5 mm to (164.0, 114.0), turned to 90 degrees
- moved C21 41.4 mm to (160.5, 118.5)
- moved C28 35.9 mm to (132.0, 147.0)
- moved C6 35.9 mm to (126.5, 147.0)
- moved R10 35.9 mm to (132.0, 151.0)
- moved R11 35.9 mm to (132.0, 149.0)
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Routing:
- net +5V: track 0.00 -> 71.3 mm
- net /Contactors/HVIL_FILTERED: track 0.00 -> 59.2 mm
- net GND: track 0.00 -> 31.5 mm, vias 0 -> 13
- net +3.3V: track 0.00 -> 23.4 mm, vias 0 -> 3
- net /Slave Power/SLAVE_5V: track 0.00 -> 19.5 mm
- net Net-(U4-FB): track 0.00 -> 18.0 mm
- net +12V: track 0.00 -> 15.6 mm
- net /CAN/CAN2_HIGH: track 0.00 -> 12.5 mm
- net /Contactors/HVIL: track 0.00 -> 12.1 mm
- net /CAN/CAN1_HIGH: track 0.00 -> 11.0 mm
- net /CAN/CAN1_LOW: track 0.00 -> 10.8 mm
- net /Power/VIN: track 0.00 -> 9.60 mm
- net /CAN/CAN2_LOW: track 0.00 -> 8.77 mm
- net Net-(U3-CANL): track 0.00 -> 7.05 mm
- net Net-(U2-CANL): track 0.00 -> 7.05 mm
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- added copper zone on In2.Cu, net +3.3V
- added copper zone on In1.Cu, net GND
Other:
- board outline added: 80 x 60 mm

Commit message: Worked on BMS master layout
Parts:
- moved JP1 95.0 mm to (145.5, 120.5)
- moved C7 87.5 mm to (122.0, 94.2), turned to 180 degrees
- moved C16 79.1 mm to (162.4, 129.5)
- moved R3 79.1 mm to (162.9, 126.4)
- moved C6 57.3 mm to (129.1, 89.8)
- moved R4 57.3 mm to (129.1, 93.8)
- moved R5 57.3 mm to (129.1, 91.8)
- moved C28 57.3 mm to (132.8, 89.8), turned to 0 degrees
- moved R10 57.3 mm to (132.8, 93.8), turned to 180 degrees
- moved R11 57.3 mm to (132.8, 91.8), turned to 0 degrees
- moved R9 54.2 mm to (145.5, 123.2)
- moved R8 34.3 mm to (154.8, 94.8), turned to -90 degrees
- moved JP3 12.9 mm to (147.2, 128.3), turned to 90 degrees
- moved J6 5.25 mm to (154.2, 128.5)
- moved C17 3.91 mm to (152.0, 103.8), turned to 180 degrees
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Connections:
- U1 pad 16: /MCU/LED -> unconnected-(U1-PB0-Pad16)
- U1 pad 17: /MCU/PRIMARY -> unconnected-(U1-PB1-Pad17)
- U1 pad 25: /CAN/CAN2_STB -> unconnected-(U1-PB11-Pad25)
- U1 pad 26: /CAN/CAN2_RX -> /CAN/CAN1_RX
- U1 pad 27: /CAN/CAN2_TX -> /CAN/CAN1_TX
- U1 pad 28: unconnected-(U1-PB14-Pad28) -> /CAN/CAN1_STB
- U1 pad 3: unconnected-(U1-PC14-Pad3) -> /MCU/LED
- U1 pad 30: unconnected-(U1-PA8-Pad30) -> /MCU/PRIMARY
- U1 pad 32: /CAN/CAN1_STB -> /CAN/CAN2_STB
- U1 pad 33: /CAN/CAN1_RX -> /CAN/CAN2_RX
- U1 pad 34: /CAN/CAN1_TX -> /CAN/CAN2_TX
Routing:
- net /CAN/CAN2_RX: track 0.00 -> 57.8 mm, vias 0 -> 2
- net /CAN/CAN2_TX: track 0.00 -> 53.9 mm, vias 0 -> 2
- net /MCU/ENABLE_SLAVES: track 5.15 -> 55.4 mm, vias 0 -> 2
- net /CAN/CAN2_STB: track 0.00 -> 47.6 mm
- net /CAN/CAN1_RX: track 0.00 -> 36.7 mm
- net /CAN/CAN1_TX: track 0.00 -> 35.9 mm, vias 0 -> 2
- net /CAN/CAN1_STB: track 0.00 -> 32.9 mm
- net GND: track 31.5 -> 58.9 mm, vias 13 -> 39
- net /Contactors/HVIL_FILTERED: track 59.2 -> 77.8 mm
- net /MCU/NRST: track 0.00 -> 15.8 mm, vias 0 -> 2
- net /Contactors/CONTACTOR_POS-: track 0.00 -> 15.3 mm
- net +3.3V: track 23.4 -> 37.8 mm, vias 3 -> 7
- net /MCU/DBG_RX: track 0.00 -> 14.3 mm
- net +12V: track 15.6 -> 28.5 mm
- net /Contactors/CONTACTOR_PRECHARGE-: track 0.00 -> 12.5 mm
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