File: hardware/aphid-vehicle-controller/monitor.kicad_sch (KiCad schematic)
At the start: 17 parts, among them J4 MONITOR_SWD, U7 STM32G431KBTx, Y2 8 MHz

Commit message: Some cleaning up
Parts:
- JP2: footprint (none) -> Jumper:SolderJumper-3_P1.3mm_Bridged12_RoundedPad1.0x1.5mm
Changed lines of the file:
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@@
 			)
 		)
-		(property "Footprint" ""
+		(property "Footprint" "Jumper:SolderJumper-3_P1.3mm_Bridged12_RoundedPad1.0x1.5mm"
 			(at 29.21 106.68 0)
 			(effects
